File: value_split/Modified/value_split.kicad_sch (KiCad schematic)
At the start: 6 parts

Commit message: KiBot generated updated
Parts:
- L1: value 3,3 nH -> 3.3 nH
Changed lines of the file:
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@@
       (effects (font (size 1.27 1.27)) (justify left))
     )
-    (property "Value" "3,3 nH" (id 1) (at 77.597 81.1784 0)
+    (property "Value" "3.3 nH" (id 1) (at 77.597 81.1784 0)
       (effects (font (size 1.27 1.27)) (justify left))
     )
@@
     )
     (path "/00000000-0000-0000-0000-0000645261a6"
-      (reference "L1") (unit 1) (value "3,3 nH") (footprint "")
+      (reference "L1") (unit 1) (value "3.3 nH") (footprint "")
     )
     (path "/00000000-0000-0000-0000-0000645266d9"
